Commit message: omni-v0.0.3

File: rl_control_new/config/urdf_folder/urdf/tiangong2.0_pro_urdf.urdf (robot description, URDF)
Before this commit: robot tiangong2pro_urdf, 37 links, 36 joints
Links:
- link ankle_pitch_l_link: geometry collision mesh filename=/home/ubuntu/omni_ws/src/Deploy_Tienkung_Pro/rl_control_new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; visual mesh filename=/home/ubuntu/omni_ws/src/Deploy_Tienkung_Pro/rl_control_new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
- link ankle_pitch_r_link: geometry collision mesh filename=/home/ubuntu/omni_ws/src/Deploy_Tienkung_Pro/rl_control_new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; visual mesh filename=/home/ubuntu/omni_ws/src/Deploy_Tienkung_Pro/rl_control_new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
- link ankle_roll_l_link: geometry collision mesh filename=/home/ubuntu/omni_ws/src/Deploy_Tienkung_Pro/rl_control_new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; visual mesh filename=/home/ubuntu/omni_ws/src/Deploy_Tienkung_Pro/rl_control_new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
- link ankle_roll_r_link: geometry collision mesh filename=/home/ubuntu/omni_ws/src/Deploy_Tienkung_Pro/rl_control_new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; visual mesh filename=/home/ubuntu/omni_ws/src/Deploy_Tienkung_Pro/rl_control_new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
- link body_yaw_link: geometry collision mesh filename=/home/ubuntu/omni_ws/src/Deploy_Tienkung_Pro/rl_control_new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; visual mesh filename=/home/ubuntu/omni_ws/src/Deploy_Tienkung_Pro/rl_control_new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
- link camera_body_back_link: geometry collision mesh filename=/home/ubuntu/omni_ws/src/Deploy_Tienkung_Pro/rl_control_new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; visual mesh filename=/home/ubuntu/omni_ws/src/Deploy_Tienkung_Pro/rl_control_new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
- link camera_body_front_link: geometry collision mesh filename=/home/ubuntu/omni_ws/src/Deploy_Tienkung_Pro/rl_control_new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; visual mesh filename=/home/ubuntu/omni_ws/src/Deploy_Tienkung_Pro/rl_control_new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
- link camera_head_link: geometry collision mesh filename=/home/ubuntu/omni_ws/src/Deploy_Tienkung_Pro/rl_control_new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; visual mesh filename=/home/ubuntu/omni_ws/src/Deploy_Tienkung_Pro/rl_control_new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
- link elbow_pitch_l_link: geometry collision mesh filename=/home/ubuntu/omni_ws/src/Deploy_Tienkung_Pro/rl_control_new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; visual mesh filename=/home/ubuntu/omni_ws/src/Deploy_Tienkung_Pro/rl_control_new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
- link elbow_pitch_r_link: geometry collision mesh filename=/home/ubuntu/omni_ws/src/Deploy_Tienkung_Pro/rl_control_new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; visual mesh filename=/home/ubuntu/omni_ws/src/Deploy_Tienkung_Pro/rl_control_new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
- link elbow_yaw_l_link: geometry collision mesh filename=/home/ubuntu/omni_ws/src/Deploy_Tienkung_Pro/rl_control_new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; visual mesh filename=/home/ubuntu/omni_ws/src/Deploy_Tienkung_Pro/rl_control_new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
- link elbow_yaw_r_link: geometry collision mesh filename=/home/ubuntu/omni_ws/src/Deploy_Tienkung_Pro/rl_control_new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; visual mesh filename=/home/ubuntu/omni_ws/src/Deploy_Tienkung_Pro/rl_control_new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
- link head_pitch_link: geometry collision mesh filename=/home/ubuntu/omni_ws/src/Deploy_Tienkung_Pro/rl_control_new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; visual mesh filename=/home/ubuntu/omni_ws/src/Deploy_Tienkung_Pro/rl_control_new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
- link head_roll_link: geometry collision mesh filename=/home/ubuntu/omni_ws/src/Deploy_Tienkung_Pro/rl_control_new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; visual mesh filename=/home/ubuntu/omni_ws/src/Deploy_Tienkung_Pro/rl_control_new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
- link head_yaw_link: geometry collision mesh filename=/home/ubuntu/omni_ws/src/Deploy_Tienkung_Pro/rl_control_new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; visual mesh filename=/home/ubuntu/omni_ws/src/Deploy_Tienkung_Pro/rl_control_new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
- link hip_pitch_l_link: geometry collision mesh filename=/home/ubuntu/omni_ws/src/Deploy_Tienkung_Pro/rl_control_new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; visual mesh filename=/home/ubuntu/omni_ws/src/Deploy_Tienkung_Pro/rl_control_new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
- link hip_pitch_r_link: geometry collision mesh filename=/home/ubuntu/omni_ws/src/Deploy_Tienkung_Pro/rl_control_new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; visual mesh filename=/home/ubuntu/omni_ws/src/Deploy_Tienkung_Pro/rl_control_new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
- link hip_roll_l_link: geometry collision mesh filename=/home/ubuntu/omni_ws/src/Deploy_Tienkung_Pro/rl_control_new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; visual mesh filename=/home/ubuntu/omni_ws/src/Deploy_Tienkung_Pro/rl_control_new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
- link hip_roll_r_link: geometry collision mesh filename=/home/ubuntu/omni_ws/src/Deploy_Tienkung_Pro/rl_control_new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; visual mesh filename=/home/ubuntu/omni_ws/src/Deploy_Tienkung_Pro/rl_control_new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
- link hip_yaw_l_link: geometry collision mesh filename=/home/ubuntu/omni_ws/src/Deploy_Tienkung_Pro/rl_control_new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; visual mesh filename=/home/ubuntu/omni_ws/src/Deploy_Tienkung_Pro/rl_control_new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
- link hip_yaw_r_link: geometry collision mesh filename=/home/ubuntu/omni_ws/src/Deploy_Tienkung_Pro/rl_control_new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; visual mesh filename=/home/ubuntu/omni_ws/src/Deploy_Tienkung_Pro/rl_control_new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
- link imu_link: geometry collision mesh filename=/home/ubuntu/omni_ws/src/Deploy_Tienkung_Pro/rl_control_new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; visual mesh filename=/home/ubuntu/omni_ws/src/Deploy_Tienkung_Pro/rl_control_new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
- link knee_pitch_l_link: geometry collision mesh filename=/home/ubuntu/omni_ws/src/Deploy_Tienkung_Pro/rl_control_new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; visual mesh filename=/home/ubuntu/omni_ws/src/Deploy_Tienkung_Pro/rl_control_new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
- link knee_pitch_r_link: geometry collision mesh filename=/home/ubuntu/omni_ws/src/Deploy_Tienkung_Pro/rl_control_new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; visual mesh filename=/home/ubuntu/omni_ws/src/Deploy_Tienkung_Pro/rl_control_new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
- link left_tcp_link: geometry collision mesh filename=/home/ubuntu/omni_ws/src/Deploy_Tienkung_Pro/rl_control_new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; visual mesh filename=/home/ubuntu/omni_ws/src/Deploy_Tienkung_Pro/rl_control_new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
- link pelvis: geometry collision mesh filename=/home/ubuntu/omni_ws/src/Deploy_Tienkung_Pro/rl_control_new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; visual mesh filename=/home/ubuntu/omni_ws/src/Deploy_Tienkung_Pro/rl_control_new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
- link right_tcp_link: geometry collision mesh filename=/home/ubuntu/omni_ws/src/Deploy_Tienkung_Pro/rl_control_new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; visual mesh filename=/home/ubuntu/omni_ws/src/Deploy_Tienkung_Pro/rl_control_new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
- link shoulder_pitch_l_link: geometry collision mesh filename=/home/ubuntu/omni_ws/src/Deploy_Tienkung_Pro/rl_control_new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; visual mesh filename=/home/ubuntu/omni_ws/src/Deploy_Tienkung_Pro/rl_control_new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
- link shoulder_pitch_r_link: geometry collision mesh filename=/home/ubuntu/omni_ws/src/Deploy_Tienkung_Pro/rl_control_new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; visual mesh filename=/home/ubuntu/omni_ws/src/Deploy_Tienkung_Pro/rl_control_new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
- link shoulder_roll_l_link: geometry collision mesh filename=/home/ubuntu/omni_ws/src/Deploy_Tienkung_Pro/rl_control_new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; visual mesh filename=/home/ubuntu/omni_ws/src/Deploy_Tienkung_Pro/rl_control_new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
- link shoulder_roll_r_link: geometry collision mesh filename=/home/ubuntu/omni_ws/src/Deploy_Tienkung_Pro/rl_control_new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; visual mesh filename=/home/ubuntu/omni_ws/src/Deploy_Tienkung_Pro/rl_control_new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
- link shoulder_yaw_l_link: geometry collision mesh filename=/home/ubuntu/omni_ws/src/Deploy_Tienkung_Pro/rl_control_new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; visual mesh filename=/home/ubuntu/omni_ws/src/Deploy_Tienkung_Pro/rl_control_new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
- link shoulder_yaw_r_link: geometry collision mesh filename=/home/ubuntu/omni_ws/src/Deploy_Tienkung_Pro/rl_control_new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; visual mesh filename=/home/ubuntu/omni_ws/src/Deploy_Tienkung_Pro/rl_control_new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
- link wrist_pitch_l_link: geometry collision mesh filename=/home/ubuntu/omni_ws/src/Deploy_Tienkung_Pro/rl_control_new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; visual mesh filename=/home/ubuntu/omni_ws/src/Deploy_Tienkung_Pro/rl_control_new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
- link wrist_pitch_r_link: geometry collision mesh filename=/home/ubuntu/omni_ws/src/Deploy_Tienkung_Pro/rl_control_new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; visual mesh filename=/home/ubuntu/omni_ws/src/Deploy_Tienkung_Pro/rl_control_new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
- link wrist_roll_l_link: geometry collision mesh filename=/home/ubuntu/omni_ws/src/Deploy_Tienkung_Pro/rl_control_new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; visual mesh filename=/home/ubuntu/omni_ws/src/Deploy_Tienkung_Pro/rl_control_new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
- link wrist_roll_r_link: geometry collision mesh filename=/home/ubuntu/omni_ws/src/Deploy_Tienkung_Pro/rl_control_new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; visual mesh filename=/home/ubuntu/omni_ws/src/Deploy_Tienkung_Pro/rl_control_new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
